File: WizLite PCB/WizLite.kicad_pcb (KiCad board)
At the start: 2 copper layers, 56 x 71 mm, 156 parts, among them J1 USB_C_Receptacle_USB2.0_16P, SW1 SW_Push, SW2 SW_Push, SW3 SW_Push, SW4 SW_Push, SW5 SW_Push, SW6 SW_Push, SW7 SW_Push, SW8 SW_Push, SW9 SW_Push, U1 CH552G, U10 XL-0807RGBC-WS2812B-S, U100 XL-0807RGBC-WS2812B-S, U101 XL-0807RGBC-WS2812B-S, U102 XL-0807RGBC-WS2812B-S, U103 XL-0807RGBC-WS2812B-S, U104 XL-0807RGBC-WS2812B-S, U105 XL-0807RGBC-WS2812B-S, U106 XL-0807RGBC-WS2812B-S, U107 XL-0807RGBC-WS2812B-S, U108 XL-0807RGBC-WS2812B-S, U109 XL-0807RGBC-WS2812B-S, U11 XL-0807RGBC-WS2812B-S, U110 XL-0807RGBC-WS2812B-S, U111 XL-0807RGBC-WS2812B-S, U112 XL-0807RGBC-WS2812B-S, U113 XL-0807RGBC-WS2812B-S, U114 XL-0807RGBC-WS2812B-S, U115 XL-0807RGBC-WS2812B-S, U116 XL-0807RGBC-WS2812B-S, U117 XL-0807RGBC-WS2812B-S, U118 XL-0807RGBC-WS2812B-S, U119 XL-0807RGBC-WS2812B-S, U12 XL-0807RGBC-WS2812B-S, U120 XL-0807RGBC-WS2812B-S, U121 XL-0807RGBC-WS2812B-S, U122 XL-0807RGBC-WS2812B-S, U123 XL-0807RGBC-WS2812B-S, U124 XL-0807RGBC-WS2812B-S, U125 XL-0807RGBC-WS2812B-S, U126 XL-0807RGBC-WS2812B-S, U127 XL-0807RGBC-WS2812B-S, U13 XL-0807RGBC-WS2812B-S, U14 XL-0807RGBC-WS2812B-S, U15 XL-0807RGBC-WS2812B-S, U16 XL-0807RGBC-WS2812B-S, U17 XL-0807RGBC-WS2812B-S, U18 XL-0807RGBC-WS2812B-S, U19 XL-0807RGBC-WS2812B-S, U2 XL-0807RGBC-WS2812B-S, U20 XL-0807RGBC-WS2812B-S, U21 XL-0807RGBC-WS2812B-S, U22 XL-0807RGBC-WS2812B-S, U23 XL-0807RGBC-WS2812B-S, U24 XL-0807RGBC-WS2812B-S, U25 XL-0807RGBC-WS2812B-S, U26 XL-0807RGBC-WS2812B-S, U27 XL-0807RGBC-WS2812B-S, U28 XL-0807RGBC-WS2812B-S, U29 XL-0807RGBC-WS2812B-S, U3 XL-0807RGBC-WS2812B-S, U30 XL-0807RGBC-WS2812B-S, U31 XL-0807RGBC-WS2812B-S, U32 XL-0807RGBC-WS2812B-S, U33 XL-0807RGBC-WS2812B-S, U34 XL-0807RGBC-WS2812B-S, U35 XL-0807RGBC-WS2812B-S, U36 XL-0807RGBC-WS2812B-S, U37 XL-0807RGBC-WS2812B-S, U38 XL-0807RGBC-WS2812B-S, U39 XL-0807RGBC-WS2812B-S, U4 XL-0807RGBC-WS2812B-S, U40 XL-0807RGBC-WS2812B-S, U41 XL-0807RGBC-WS2812B-S, U42 XL-0807RGBC-WS2812B-S, U43 XL-0807RGBC-WS2812B-S, U44 XL-0807RGBC-WS2812B-S, U45 XL-0807RGBC-WS2812B-S, U46 XL-0807RGBC-WS2812B-S, U47 XL-0807RGBC-WS2812B-S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

Commit message: Added PCB Art & Added Production Files
Parts:
- added C3: 47uF, Capacitor_SMD:C_1210_3225Metric_Pad1.33x2.70mm_HandSolder, F.Cu at (37.5, 81.0)
- added C4: 47uF, Capacitor_SMD:C_1210_3225Metric_Pad1.33x2.70mm_HandSolder, F.Cu at (37.5, 48.0)
- added G***: LOGO, LOGO, F.Cu at (42.7, 90.7)
- added G***: LOGO, LOGO, F.Cu at (70.8, 90.4)
- added G***: LOGO, LOGO, B.Cu at (57.1, 63.3)
Routing:
- net +5V: track 587.3 -> 595.6 mm, vias 132 -> 134
- net +3V3: track 212.9 -> 216.3 mm
- net GND: vias 181 -> 182
Other:
- board text added: "ABean :)"
- board text added: "Boot"
- board text added: "Player 1"
- board text added: "Player 2"
- board text added: "Wiz-Lite"
